File: rpi-cc2538-uart.brd (EAGLE design)
At the start: 48.5 x 23 mm, 10 parts

Commit message: Add files via upload
Parts:
- removed U$4: (no value), SparkFun-Aesthetics:OSHW-LOGO-L
- U$1: device codm:CC2538-CN -> CC2538-CN:CC2538-CN
- U$2: device codm:CODM-LOGO -> logo_flobul:LOGO_FLOBUL_2MM
- moved U$2 18.0 mm to (46.0, 1.00)
- moved U$3 2.24 mm to (20.0, 3.00)
Connections:
- net GND: no longer U$1.GND@2
Routing:
- net RXD: track 29.3 -> 23.9 mm
- net TMS: track 29.5 -> 33.1 mm
- net TCK: track 28.7 -> 32.2 mm
- net VCC: track 36.5 -> 39.6 mm
- net TXD: track 30.1 -> 27.1 mm
- net TDO: track 27.7 -> 30.7 mm
- net TDI: track 27.2 -> 28.5 mm
Other:
- board text removed: "90083-0.4"
- board text removed: "90083-0.4 CC-BY-SA-NC"
- board text removed: "CC2538-LR RPi Serial Module V0.4 with integrated CC2592 PA/LNA codm.de, (c) 2020"
- board text removed: "codm.de"
