File: rpi-cc2538-uart.sch (EAGLE design)
At the start: 7 parts

Commit message: Add files via upload
Parts:
- U$1: device codm:CC2538-CN -> CC2538-CN:CC2538-CN
Other:
- note added: "cod.m GmbH, 2020 https://www.codm.de Modified by Flobul, 2023 CC-BY-SA-NC"
- note removed: "cod.m GmbH, 2020 https://www.codm.de CC-BY-SA-NC"
- moved on the sheet: C1, R1
Changed lines of the file:
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@@
 <drawing>
 <settings>
-<setting alwaysvectorfont="yes"/>
+<setting alwaysvectorfont="no"/>
 <setting verticaltext="up"/>
 </settings>
@@
 </classes>
 <parts>
-<part name="U$1" library="codm" library_urn="urn:adsk.eagle:library:11602856" deviceset="CC2538-CN" device="" package3d_urn="urn:adsk.eagle:package:21916107/5"/>
+<part name="U$1" library="CC2538-CN" deviceset="CC2538-CN" device="" package3d_urn="urn:adsk.eagle:package:21916107/4"/>
 <part name="JP1" library="pinhead" deviceset="PINHD-2X5" device="" override_package3d_urn="urn:adsk.eagle:package:22254121/2" override_package_urn="urn:adsk.eagle:footprint:22254122/1"/>
 <part name="C1" library="rcl" library_urn="urn:adsk.eagle:library:334" deviceset="CPOL-EU" device="A/3216-18W" package3d_urn="urn:adsk.eagle:package:23408/2" override_package3d_urn="urn:adsk.eagle:package:22254313/2" override_package_urn="urn:adsk.eagle:footprint:22913/1" value="33u"/>
@@
 <sheet>
 <plain>
-<text x="185.42" y="-5.08" size="2.54" layer="94">cod.m GmbH, 2020
+<text x="185.42" y="-7.62" size="2.54" layer="94">cod.m GmbH, 2020
 https://www.codm.de
+Modified by Flobul, 2023
 CC-BY-SA-NC</text>
 </plain>
@@
 <attribute name="VALUE" x="184.15" y="38.1" size="1.778" layer="96"/>
 </instance>
-<instance part="C1" gate="G$1" x="55.88" y="83.82" smashed="yes" rot="R180">
-<attribute name="NAME" x="54.356" y="83.439" size="1.778" layer="95" rot="R180"/>
-<attribute name="VALUE" x="54.356" y="88.519" size="1.778" layer="96" rot="R180"/>
-</instance>
-<instance part="R1" gate="G$1" x="154.94" y="99.06" smashed="yes" rot="R90">
-<attribute name="NAME" x="153.4414" y="95.25" size="1.778" layer="95" rot="R90"/>
-<attribute name="VALUE" x="158.242" y="95.25" size="1.778" layer="96" rot="R90"/>
+<instance part="C1" gate="G$1" x="88.9" y="116.84" smashed="yes" rot="R180">
+<attribute name="NAME" x="87.376" y="116.459" size="1.778" layer="95" rot="R180"/>
+<attribute name="VALUE" x="87.376" y="121.539" size="1.778" layer="96" rot="R180"/>
+</instance>
+<instance part="R1" gate="G$1" x="160.02" y="96.52" smashed="yes">
+<attribute name="NAME" x="156.21" y="98.0186" size="1.778" layer="95"/>
+<attribute name="VALUE" x="156.21" y="93.218" size="1.778" layer="96"/>
 </instance>
 <instance part="JTAG" gate="G$1" x="195.58" y="111.76" smashed="yes">
@@
 <segment>
 <pinref part="U$1" gate="G$1" pin="VCC"/>
-<wire x1="96.52" y1="88.9" x2="60.96" y2="88.9" width="0.1524" layer="91"/>
-<wire x1="60.96" y1="88.9" x2="60.96" y2="78.74" width="0.1524" layer="91"/>
-<wire x1="60.96" y1="78.74" x2="55.88" y2="78.74" width="0.1524" layer="91"/>
+<wire x1="96.52" y1="96.52" x2="88.9" y2="96.52" width="0.1524" layer="91"/>
 <pinref part="C1" gate="G$1" pin="+"/>
-<wire x1="55.88" y1="78.74" x2="48.26" y2="78.74" width="0.1524" layer="91"/>
-<wire x1="55.88" y1="81.28" x2="55.88" y2="78.74" width="0.1524" layer="91"/>
-<junction x="55.88" y="78.74"/>
-<label x="48.26" y="78.74" size="1.27" layer="95" rot="R180" xref="yes"/>
+<wire x1="88.9" y1="96.52" x2="83.82" y2="96.52" width="0.1524" layer="91"/>
+<wire x1="88.9" y1="114.3" x2="88.9" y2="96.52" width="0.1524" layer="91"/>
+<junction x="88.9" y="96.52"/>
+<label x="83.82" y="96.52" size="1.27" layer="95" rot="R180" xref="yes"/>
 </segment>
 <segment>
 <pinref part="R1" gate="G$1" pin="2"/>
-<wire x1="154.94" y1="104.14" x2="154.94" y2="109.22" width="0.1524" layer="91"/>
-<label x="154.94" y="109.22" size="1.27" layer="95" rot="R90" xref="yes"/>
+<wire x1="165.1" y1="96.52" x2="175.26" y2="96.52" width="0.1524" layer="91"/>
+<label x="175.26" y="96.52" size="1.27" layer="95" rot="R90" xref="yes"/>
 </segment>
 <segment>
@@
 <segment>
 <pinref part="U$1" gate="G$1" pin="GND"/>
-<wire x1="96.52" y1="91.44" x2="55.88" y2="91.44" width="0.1524" layer="91"/>
-<label x="48.26" y="91.44" size="1.27" layer="95" rot="R180" xref="yes"/>
+<wire x1="147.32" y1="99.06" x2="147.32" y2="121.92" width="0.1524" layer="91"/>
+<label x="147.32" y="129.54" size="1.27" layer="95" rot="R180" xref="yes"/>
 <pinref part="C1" gate="G$1" pin="-"/>
-<wire x1="55.88" y1="91.44" x2="48.26" y2="91.44" width="0.1524" layer="91"/>
-<wire x1="55.88" y1="88.9" x2="55.88" y2="91.44" width="0.1524" layer="91"/>
-<junction x="55.88" y="91.44"/>
+<wire x1="147.32" y1="121.92" x2="147.32" y2="129.54" width="0.1524" layer="91"/>
+<wire x1="88.9" y1="121.92" x2="147.32" y2="121.92" width="0.1524" layer="91"/>
+<junction x="147.32" y="121.92"/>
 </segment>
 <segment>
@@
 <segment>
 <pinref part="U$1" gate="G$1" pin="PA0"/>
-<wire x1="147.32" y1="66.04" x2="162.56" y2="66.04" width="0.1524" layer="91"/>
-<label x="162.56" y="66.04" size="1.27" layer="95" xref="yes"/>
+<wire x1="132.08" y1="58.42" x2="132.08" y2="43.18" width="0.1524" layer="91"/>
+<label x="132.08" y="43.18" size="1.27" layer="95" xref="yes"/>
 </segment>
 </net>
@@
 <segment>
 <pinref part="U$1" gate="G$1" pin="PA1"/>
-<wire x1="147.32" y1="68.58" x2="162.56" y2="68.58" width="0.1524" layer="91"/>
-<label x="162.56" y="68.58" size="1.27" layer="95" xref="yes"/>
+<wire x1="134.62" y1="58.42" x2="134.62" y2="45.72" width="0.1524" layer="91"/>
+<label x="134.62" y="45.72" size="1.27" layer="95" xref="yes"/>
 </segment>
 </net>
@@
 <wire x1="147.32" y1="91.44" x2="154.94" y2="91.44" width="0.1524" layer="91"/>
 <pinref part="R1" gate="G$1" pin="1"/>
-<wire x1="154.94" y1="93.98" x2="154.94" y2="91.44" width="0.1524" layer="91"/>
+<wire x1="154.94" y1="96.52" x2="154.94" y2="91.44" width="0.1524" layer="91"/>
 <junction x="154.94" y="91.44"/>
 <wire x1="154.94" y1="91.44" x2="180.34" y2="91.44" width="0.1524" layer="91"/>
@@
 <segment>
 <pinref part="U$1" gate="G$1" pin="TMS"/>
-<wire x1="96.52" y1="86.36" x2="86.36" y2="86.36" width="0.1524" layer="91"/>
-<label x="86.36" y="86.36" size="1.27" layer="95" rot="R180" xref="yes"/>
+<wire x1="96.52" y1="91.44" x2="86.36" y2="91.44" width="0.1524" layer="91"/>
+<label x="86.36" y="91.44" size="1.27" layer="95" rot="R180" xref="yes"/>
 </segment>
 <segment>
@@
 <segment>
 <pinref part="U$1" gate="G$1" pin="TCK"/>
-<wire x1="96.52" y1="83.82" x2="86.36" y2="83.82" width="0.1524" layer="91"/>
-<label x="86.36" y="83.82" size="1.27" layer="95" rot="R180" xref="yes"/>
+<wire x1="96.52" y1="88.9" x2="86.36" y2="88.9" width="0.1524" layer="91"/>
+<label x="86.36" y="88.9" size="1.27" layer="95" rot="R180" xref="yes"/>
 </segment>
 <segment>
@@
 <segment>
 <pinref part="U$1" gate="G$1" pin="PB7"/>
-<wire x1="96.52" y1="81.28" x2="86.36" y2="81.28" width="0.1524" layer="91"/>
-<label x="86.36" y="81.28" size="1.27" layer="95" rot="R180" xref="yes"/>
+<wire x1="96.52" y1="86.36" x2="86.36" y2="86.36" width="0.1524" layer="91"/>
+<label x="86.36" y="86.36" size="1.27" layer="95" rot="R180" xref="yes"/>
 </segment>
 <segment>
@@
 <segment>
 <pinref part="U$1" gate="G$1" pin="PB6"/>
-<wire x1="96.52" y1="78.74" x2="86.36" y2="78.74" width="0.1524" layer="91"/>
-<label x="86.36" y="78.74" size="1.27" layer="95" rot="R180" xref="yes"/>
-</segment>
-<segment>
+<wire x1="96.52" y1="83.82" x2="86.36" y2="83.82" width="0.1524" layer="91"/>
+<label x="86.36" y="83.82" size="1.27" layer="95" rot="R180" xref="yes"/>
+</segment>
+<segment>
